File: Improved LoRa Camera/PCB Files/ESP32S3 LoRa Mini Camera Board 120426/ESP32S3 LoRa Mini Camera Board 120426.brd (EAGLE design)
At the start: 75 x 40 mm, 54 parts, among them IC1 RFM98_PIH, IC2 ESP32S3_DEVKIT, IC3 INA219, IC4 FM24CL64, Q1 BC547INLINE

Commit message: Add LR2021
Changed lines of the file:
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@@
 <text x="27.6921" y="26.9123" size="1" layer="26" font="vector" ratio="15" rot="SMR270">R2</text>
 <text x="27.7221" y="22.3523" size="1" layer="26" font="vector" ratio="15" rot="SMR270">C3</text>
-<text x="23.5677" y="20.5821" size="1.778" layer="25" font="vector" ratio="15">+</text>
+<text x="23.5677" y="20.5821" size="1.778" layer="26" font="vector" ratio="15">+</text>
 <text x="30.9379" y="20.8177" size="1.778" layer="25" font="vector" ratio="15" rot="R90">-</text>
 <text x="27.7021" y="17.5723" size="1" layer="26" font="vector" ratio="15" rot="SMR270">R3</text>
